File: snowflake.kicad_pcb (KiCad board)
At the start: 2 copper layers, 19 x 19 mm, 21 parts, among them J1 USB_C_Receptacle_USB2.0_14P, SW1 SW_Push, SW2 DFU, U1 CH552E

Commit message: update
Routing:
- net GND: vias 16 -> 23
Changed lines of the file:
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@@
+	)
+	(via
+		(at 97.68 94.35)
+		(size 0.6)
+		(drill 0.3)
+		(layers "F.Cu" "B.Cu")
+		(free yes)
+		(net 2)
+	)
+	(via
+		(at 99.72 77)
+		(size 0.6)
+		(drill 0.3)
+		(layers "F.Cu" "B.Cu")
+		(free yes)
+		(net 2)
 	)
 	(via
@@
 	)
 	(via
+		(at 100.7 89.06)
+		(size 0.6)
+		(drill 0.3)
+		(layers "F.Cu" "B.Cu")
+		(free yes)
+		(net 2)
+	)
+	(via
+		(at 90.21 78.53)
+		(size 0.6)
+		(drill 0.3)
+		(layers "F.Cu" "B.Cu")
+		(free yes)
+		(net 2)
+	)
+	(via
 		(at 96.55 87.5)
 		(size 0.6)
 		(drill 0.3)
 		(layers "F.Cu" "B.Cu")
+		(net 2)
+	)
+	(via
+		(at 104.31 94.28)
+		(size 0.6)
+		(drill 0.3)
+		(layers "F.Cu" "B.Cu")
+		(free yes)
 		(net 2)
 	)
@@
 	)
 	(via
+		(at 92.73 80.03)
+		(size 0.6)
+		(drill 0.3)
+		(layers "F.Cu" "B.Cu")
+		(free yes)
+		(net 2)
+	)
+	(via
 		(at 95.85 76.8)
 		(size 0.6)
 		(drill 0.3)
+		(layers "F.Cu" "B.Cu")
+		(free yes)
+		(net 2)
+	)
+	(via
+		(at 108.17 91.96)
+		(size 0.6)
+		(drill 0.3)
