File: pcb/snowflake.kicad_pcb (KiCad board)
At the start: 2 copper layers, 19 x 19 mm, 21 parts, among them J1 USB_C_Receptacle_USB2.0_14P, SW1 SW_Push, SW2 DFU, U1 CH552E

Commit message: clean up repo
Parts:
- moved U1 0.37 mm to (101.3, 90.9)
- moved R4 0.36 mm to (96.6, 92.1)
Routing:
- net +5V: track 35.4 -> 35.9 mm
- net GND: track 15.3 -> 15.0 mm, vias 23 -> 22
